File: BLDC.sch (EAGLE design)
At the start: 119 parts, among them J1 J_1X4, J2 J_1X6, J3 J_1X7, J7 1-770178-0, J8 1-770174-1, Q1 IRFS7530TRLPBF, Q2 IRFS7530TRLPBF, Q3 IRFS7530TRLPBF, Q4 IRFS7530TRLPBF, Q5 IRFS7530TRLPBF, Q6 IRFS7530TRLPBF, U1 DRV8302, U102 LM3671MF-3.3/NOPB, U104 MCP2562, U2 STM32F405RGT6, Y1 8MHz

Commit message: renumbered parts
Parts:
- removed C109: 4.7uF, rcl:C-USC0805
- removed C115, C116: 0.1uF, rcl:C-USC0805
- removed C49: 4n7, rcl:C-USC0805
- removed C50: 2.2uf, rcl:C-USC0805
- removed L102: 2.2uH, FormE:L0805
- removed R115: 120R, rcl:R-US_R0805
- removed R47: 10K, adafruit:R-US_R0805
- removed U104: MCP2562, FormE:MCP256X-SOIC
- added C39, C48: 15uf,100V, rcl:C-USC0805
- added C41, C45: 10uf,50V, rcl:C-USC0805
- added C47: 100uf, rcl:C-USC0805
- added D1: 5V, FormE:PLVA650A
- added L2: 2.2uH, FormE:L0805
- added R43: 4.7R, adafruit:R-US_R0805
- added R45: 39k, adafruit:R-US_R0805
- added U3: DRV8302, FormE:DRV8302
- C1: value 2.2uf -> 2200uF; device rcl:C-USC0805 -> FormE:UVR1J222MHD; PARTNO GRM21BR61E106KA73L -> (none)
- C11: value 15p -> 2.2uf
- C13, C14, C15: value 4n7 -> 2.2uf
- C17: value 120pf -> 2.2uf
- C18: value 6.8n -> 2.2uf
- C2, C7: value 2.2uf -> 0.1uF; PARTNO GRM21BR61E106KA73L -> GRM21BR71E104KA01L
- C21: value 22n -> 2.2uf
- C25: value 100n -> 2.2uf
- C26: value 100uf -> 22n
- C27: value 10uf, 50V -> 2.2uf
- C28: value 220n -> 6.8n
- C29: value 220n -> 120pf
- C3, C4, C5, C6: value 2.2uf -> 4n7
- C30: value 220n -> 4.7uF; PARTNO GRM21BR61E106KA73L -> GRM21BC81E475KA12L
- C31, C32: value 2.2n -> 10uf,50V
- C35, C36, C37: value 10uf,50V -> 220n
- C38: value 15uf,100V -> 10uf, 50V
- C40: value 2200uF -> 10uf,50V; device FormE:UVR1J222MHD -> rcl:C-USC0805; PARTNO (none) -> GRM21BR61E106KA73L
- C42: value 10uf,50V -> 100n
- C43: value 10uf,50V -> 2.2n
- C44: value 15uf,100V -> 2.2n
- C9: value 2.2uf -> 15p
- J1: value J_1X4 -> 1-770174-1; device FormE:J_1X4 -> FormE:1-770174-1
- J2: value J_1X6 -> 1-770178-0; device FormE:J_1X6 -> FormE:1-770178-0
- J3: value J_1X7 -> J_1X4; device FormE:J_1X7 -> FormE:J_1X4
- J4: value (none) -> J_1X7; device FormE:J_1X2 -> FormE:J_1X7
- J5: value (none) -> J_1X6; device FormE:J_1X2 -> FormE:J_1X6
- J7: value 1-770178-0 -> (none); device FormE:1-770178-0 -> FormE:J_1X2
- J8: value 1-770174-1 -> (none); device FormE:1-770174-1 -> FormE:J_1X2
- R1: value 1k -> DNP
- R10, R26: value 2.2k -> 10k
- R12: value 2.2k -> 39K
- R14: value 220K -> 1k
- R15: value 15K -> 1k
- R16: value 18K -> 10K; device adafruit:R-US_R0805 -> FormE:NCP18XH103F03RB; PARTNO ERJ-6ENF1001V -> (none)
- R17: value 3K3 -> 10K
- R18: value 10k -> 39k
- R19: value 220K -> 2.2k
- R20, R22: value 100R -> 39k
- R21: value 1k -> 2.2k
- R23: value 100R -> 2.2k
- R24: value 100R -> 18K
- R25: value 39k -> 3K3
- R27, R29: value 39k -> 220K
- R28: value 2.2k -> 15K
- R30: value 2.2k -> 100R
- R31: value 39k -> 100R
- R32, R33: value 4.7R -> 100R
- R34: value 4.7R -> 1k
- R35: value 4.7R -> .001R; device adafruit:R-US_R0805 -> FormE:WSLP27261L000FEA; PARTNO ERJ-6ENF1001V -> (none)
- R36: value 39k -> .001R; device adafruit:R-US_R0805 -> FormE:WSLP27261L000FEA; PARTNO ERJ-6ENF1001V -> (none)
- R38: value 39k -> 4.7R
- R39: value 4.7R -> 39k
- R4: value 1k -> 120R; device adafruit:R-US_R0805 -> rcl:R-US_R0805; PARTNO ERJ-6ENF1001V -> ERJ-6ENF1200V
- R40, R41: value .001R -> 4.7R; device FormE:WSLP27261L000FEA -> adafruit:R-US_R0805; PARTNO (none) -> ERJ-6ENF1001V
- R42: value 10K -> 39k; device FormE:NCP18XH103F03RB -> adafruit:R-US_R0805; PARTNO (none) -> ERJ-6ENF1001V
- R44: value 10K -> 4.7R
- R5: value DNP -> 2.2k
- R7: value 39K -> 2.2k
- R8: value 10k -> 10K
- U1: value DRV8302 -> MCP2562; device FormE:DRV8302 -> FormE:MCP256X-SOIC; PARTNO (none) -> MCP2562FD-E/SN
- renumbered C110 to C46, D3 to D2, U102 to U4
Connections:
- net +3V3: now also C12.1, C13.1, C15.1, C16.1, C17.1, C20.1, C21.1, J2.5, J4.6, L1.P$2, LED3.A, R16.2, R5.2, R6.2, R7.2, R8.2, U1.SPLIT/VIO, U3.M_OC, U3.REF; no longer C1.1, C115.1, C3.1, C4.1, C7.1, C8.1, C9.1, J3.6, J7.5, L102.P$2, LED1.A, R10.2, R12.2, R13.2, R42.2, R47.2, U1.M_OC, U1.REF, U104.SPLIT/VIO
- net +5V: now also C30.1, C47.1, C7.1, D1.CATHODE, J3.4, J4.7, J5.6, L2.P$2, R1.1, R24.1, U1.VDD; no longer C109.1, C116.1, C26.1, J1.4, J2.6, J3.7, L1.P$2, R16.1, R5.1, U104.VDD
- net ADC_TEMP: now also C14.1, R16.1, R17.2; no longer C50.1, R42.1, R44.2
- net AN_IN: now also C8.1, R12.2, R13.1; no longer C12.1, R6.1, R7.2
- net AUX_1: now also J6.1; no longer J4.1
- net AUX_2: now also J6.2; no longer J4.2
- net AUX_3: now also J7.1; no longer J5.1
- net AUX_4: now also J7.2; no longer J5.2
- net AUX_5: now also J8.1; no longer J6.1
- net AUX_6: now also J8.2; no longer J6.2
- net BR_SO1: now also U3.SO1; no longer U1.SO1
- net BR_SO2: now also U3.SO2; no longer U1.SO2
- net CAR_CAN_N: now also J3.2, R4.1, U1.CANL; no longer J1.2, R115.1, U104.CANL
- net CAR_CAN_P: now also J3.3, R4.2, U1.CANH; no longer J1.3, R115.2, U104.CANH
- net CAR_CAN_RX: now also U1.RXD; no longer U104.RXD
- net CAR_CAN_TX: now also U1.TXD; no longer U104.TXD
- net DC_CAL: now also U3.DC_CAL; no longer U1.DC_CAL
- net DGND: now also C1.-; no longer C40.-
- net EN_GATE: now also U3.EN_GATE; no longer U1.EN_GATE
- net FAULT: now also U3.NFAULT; no longer U1.NFAULT
- net GND: now also C11.2, C21.2, C25.2, C28.2, C29.2, C30.2, C31.2, C32.2, C39.2, C40.2, C41.2, C45.2, C47.2, C48.2, C9.1, D1.ANODE, J4.1, J5.1, Q4.S, R13.2, R14.1, R15.1, R17.1, R19.1, R23.1, R25.2, R27.2, R29.2, R34.1, R35.1, R36.1, R42.2, U1.STBY, U1.VSS, U3.AGND, U3.GAIN, U3.GND, U3.M_PWM, U3.SL_B; no longer C1.2, C109.2, C11.1, C115.2, C116.2, C26.2, C35.2, C36.2, C37.2, C42.2, C43.2, C44.2, C49.2, C50.2, C9.2, J1.1, J7.1, Q5.S, R1.1, R14.2, R17.2, R18.1, R19.2, R2.1, R28.1, R30.1, R36.2, R40.1, R41.1, R44.1, R6.2, U1.AGND, U1.GAIN, U1.GND, U1.M_PWM, U1.SL_B, U104.STBY, U104.VSS
- net H1: now also U3.INH_A; no longer U1.INH_A
- net H1_LOW: now also Q2.S, R36.2, R39.2, R42.1, U3.SL_A; no longer Q4.S, R31.2, R36.1, R41.2, U1.SL_A
- net H1_VS: now also C35.2, Q1.S, Q2.D, R22.1, U3.SH_A; no longer C28.2, Q3.S, Q4.D, R29.1, U1.SH_A
- net H2: now also U3.INH_B; no longer U1.INH_B
- net H2_VS: now also C36.2, Q3.S, Q4.D, R20.1, U3.SH_B; no longer C29.2, Q1.S, Q5.D, R27.1, U1.SH_B
- net H3: now also U3.INH_C; no longer U1.INH_C
- net H3_LOW: now also R35.2, R45.2, U3.SL_C; no longer R38.2, R40.2, U1.SL_C
- net H3_VS: now also C37.2, Q5.S, R18.1, U3.SH_C; no longer C30.2, Q2.S, R25.1, U1.SH_C
- net HALL_1_IN: now also J5.5, R5.1, R6.1, R7.1; no longer J2.5, R12.1, R13.1, R8.1
- net HALL_1_OUT: now also C3.1, C4.1, C5.1, R10.2; no longer C13.1, C14.1, C15.1, R8.2
- net HALL_2_IN: now also J5.4; no longer J2.4
- net HALL_3_IN: now also J5.3; no longer J2.3
- net L1: now also U3.INL_A; no longer U1.INL_A
- net L2: now also U3.INL_B; no longer U1.INL_B
- net L3: now also U3.INL_C; no longer U1.INL_C
- net LED_GREEN: now also LED1.A; no longer LED3.A
- net MISO_ADC_EXT2: now also J4.2; no longer J3.2
- net M_H1: now also R38.1, U3.GH_A; no longer R32.1, U1.GH_A
- net M_H2: now also R41.1, U3.GH_B; no longer R33.1, U1.GH_B
- net M_H3: now also R44.1, U3.GH_C; no longer R34.1, U1.GH_C
- net M_L1: now also R37.1, R43.1, U3.GL_A; no longer R35.1, R39.1, U1.GL_A
- net M_L2: now also R40.1, U3.GL_B; no longer R37.1, U1.GL_B
- net M_L3: now also U3.GL_C; no longer U1.GL_C
- net N$1: now also R15.2; no longer R1.2
- net N$10: now also C28.1, R28.1; no longer C18.1, R15.1
- net N$11: now also L1.P$1; no longer L102.P$1
- net N$12: now also C29.1, R28.2, U3.COMP; no longer C17.1, R15.2, U1.COMP
- net N$13: now also R24.2, R25.1, U3.VSENSE; no longer R16.2, R17.1, U1.VSENSE
- net N$14: now also R26.2, U3.DTC; no longer R18.2, U1.DTC
- net N$15: now also C25.1, U3.DVDD, U3.OC_ADJ; no longer C22.1, U1.DVDD, U1.OC_ADJ
- net N$16: now also C22.1, C24.1, U3.GVDD; no longer C19.1, C20.1, U1.GVDD
- net N$17: now also C26.1, U3.CP1; no longer C21.1, U1.CP1
- net N$18: now also C27.1, U3.AVDD; no longer C24.1, U1.AVDD
- net N$19: now also C26.2, U3.CP2; no longer C21.2, U1.CP2
- net N$2: now also LED1.C, R14.2; no longer LED3.C, R2.2
- net N$20: now also C42.1, U3.BST_BK; no longer C25.1, U1.BST_BK
- net N$21: now also C42.2, L2.P$1, U3.PH, U3.PH_A; no longer C25.2, L1.P$1, U1.PH, U1.PH_A
- net N$22: now also R29.1, U3.BIAS; no longer R19.1, U1.BIAS
- net N$23: now also C35.1, U3.BST_A; no longer C28.1, U1.BST_A
- net N$24: now also C43.1, R30.1, U3.SN1; no longer C31.1, R20.1, U1.SN1
- net N$25: now also C36.1, U3.BST_B; no longer C29.1, U1.BST_B
- net N$26: now also C43.2, R31.1, U3.SP1; no longer C31.2, R22.1, U1.SP1
- net N$27: now also C37.1, U3.BST_C; no longer C30.1, U1.BST_C
- net N$28: now also C44.2, R33.1, U3.SP2; no longer C32.2, R24.1, U1.SP2
- net N$29: now also C44.1, R32.1, U3.SN2; no longer C32.1, R23.1, U1.SN2
- net N$3: now also R3.2; no longer R4.2
- net N$30: now also Q1.G, R38.2; no longer Q3.G, R32.2
- net N$31: now also Q3.G, R41.2; no longer Q1.G, R33.2
- net N$32: now also Q5.G, R44.2; no longer Q2.G, R34.2
- net N$33: now also Q2.G, R37.2, R39.1; no longer Q4.G, R31.1, R35.2
- net N$34: now also Q4.G, R40.2; no longer Q5.G, R37.2
- net N$35: now also R43.2, R45.1; no longer R38.1, R39.2
- net N$4: now also R2.2; no longer R3.2
- net N$5: now also R1.2; no longer R5.2
- net N$6: now also C18.1, C19.1; no longer C5.1, C6.1
- net N$7: now also C10.2; no longer C11.2
- net N$8: now also C9.2; no longer C10.2
- net N$81: now also LED3.C, R34.2; no longer LED1.C, R21.2
- net N$9: now also R27.1, U3.RT_CLK; no longer R14.1, U1.RT_CLK
- net NRST: now also C11.1, J2.2; no longer C16.1, J7.2
- net RX_SCL_MOSI: now also J4.5; no longer J3.5
- net SCK_ADC_EXT: now also J4.3; no longer J3.3
- net SENS1: now also R18.2, R19.2; no longer R25.2, R26.2
- net SENS2: now also R20.2, R21.2; no longer R27.2, R28.2
- net SENS3: now also R22.2, R23.2; no longer R29.2, R30.2
- net SH1_A: now also R30.2, R35.22; no longer R20.2, R40.22
- net SH1_B: now also R31.2, R35.12; no longer R22.2, R40.12
- net SH2_A: now also R32.2, R36.22; no longer R23.2, R41.22
- net SH2_B: now also R33.2, R36.12; no longer R24.2, R41.12
- net SWCLK: now also J2.4; no longer J7.4
- net SWDIO: now also J2.3; no longer J7.3
- net TEMP_IN: now also J5.2, R8.1; no longer J2.2, R47.1
- net TEMP_MOTOR: now also C6.1; no longer C49.1
- net TX_SDA_NSS: now also J4.4; no longer J3.4
- net USB_DM: now also R3.1; no longer R4.1
- net USB_DP: now also R2.1; no longer R3.1
- net VCC: now also C1.+, C31.1, C32.1, C39.1, C40.1, C41.1, C45.1, C48.1, Q5.D, U3.PVDD1, U3.PVDD2, U3.PVDD2_A; no longer C27.1, C35.1, C36.1, C37.1, C40.+, C42.1, C43.1, C44.1, Q2.D, U1.PVDD1, U1.PVDD2, U1.PVDD2_A
- net V_BATT: now also R12.1; no longer R7.1
Other:
- note removed: "DIODE!!!"
- moved on the sheet: C10, C11, C12, C13, C14, C15, C16, C17, C18, C19, C2, C20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

Commit message: updated BOM
Parts:
- C1: PARTNO (none) -> UVR1J222MHD
- D2: PARTNO (none) -> CD1206-B260
- LED2: device FormE:LEDCHIP-LED0805 -> FormE:5988110107F; PARTNO 598-8170-107F -> (none)
- Q1, Q2, Q3, Q4, Q5, Q6: PARTNO (none) -> IRFS7530TRLPBF
- R10, R11, R17, R26, R9: PARTNO ERJ-6ENF1001V -> ERJ-6ENF1002V
- R13, R19, R21, R23, R5, R6, R7: PARTNO ERJ-6ENF1001V -> ERJ-6ENF2201V
- R16: PARTNO (none) -> NCP18XH103F03RB
- R18, R20, R22, R39, R42, R45: PARTNO ERJ-6ENF1001V -> ERJ-6ENF3902V
- R24: PARTNO ERJ-6ENF1001V -> ERJ-6ENF2402V
- R25: PARTNO ERJ-6ENF1001V -> ERJ-6ENF3301V
- R27, R29: PARTNO ERJ-6ENF1001V -> ERJ-6ENF2203V
- R28: PARTNO ERJ-6ENF1001V -> ERJ-6ENF1502V
- R30, R31, R32, R33: PARTNO ERJ-6ENF1001V -> ERJ-6ENF1000V
- R37, R38, R40, R41, R43, R44: PARTNO ERJ-6ENF1001V -> ERJ-6RQF4R7V
- R8: value 10K -> 10k; PARTNO ERJ-6ENF1001V -> ERJ-6ENF1002V
- U3: PARTNO (none) -> DRV8302DCA
Other:
- note added: "r35,36"

Commit message: gate driver module progress
Changed lines of the file:
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@@
 <pinref part="U3" gate="G$1" pin="COMP"/>
 <wire x1="152.4" y1="55.88" x2="149.86" y2="55.88" width="0.1524" layer="91"/>
-<wire x1="149.86" y1="55.88" x2="147.32" y2="55.88" width="0.1524" layer="91"/>
-<wire x1="147.32" y1="99.06" x2="147.32" y2="55.88" width="0.1524" layer="91"/>
 <pinref part="C29" gate="G$1" pin="1"/>
-<wire x1="172.72" y1="81.28" x2="172.72" y2="99.06" width="0.1524" layer="91"/>
-<wire x1="172.72" y1="99.06" x2="147.32" y2="99.06" width="0.1524" layer="91"/>
+<wire x1="172.72" y1="81.28" x2="172.72" y2="96.52" width="0.1524" layer="91"/>
 <pinref part="R28" gate="G$1" pin="2"/>
 <wire x1="165.1" y1="93.98" x2="165.1" y2="96.52" width="0.1524" layer="91"/>
 <wire x1="165.1" y1="96.52" x2="149.86" y2="96.52" width="0.1524" layer="91"/>
 <wire x1="149.86" y1="96.52" x2="149.86" y2="55.88" width="0.1524" layer="91"/>
-<junction x="149.86" y="55.88"/>
+<wire x1="165.1" y1="96.52" x2="172.72" y2="96.52" width="0.1524" layer="91"/>
+<junction x="165.1" y="96.52"/>
 </segment>
 </net>

Commit message: stm32 module progress
Connections:
- net HALL_1_IN: no longer R10.1, R11.1, R6.1, R7.1
- net HALL_1_OUT: no longer C4.1, C5.1, R10.2, R11.2
- net HALL_2_IN: now also R10.1, R11.1, R6.1, R7.1
- net HALL_2_OUT: now also C4.1, R10.2
- net HALL_3_OUT: now also C5.1, R11.2
Changed lines of the file:
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@@
+</segment>
+<segment>
+<wire x1="-266.7" y1="63.5" x2="-246.38" y2="63.5" width="0.1524" layer="91"/>
+<label x="-261.62" y="63.5" size="1.778" layer="95"/>
+<pinref part="J5" gate="G$1" pin="5"/>
+</segment>
+</net>
+<net name="HALL_2_IN" class="0">
+<segment>
+<wire x1="-266.7" y1="60.96" x2="-246.38" y2="60.96" width="0.1524" layer="91"/>
+<label x="-261.62" y="60.96" size="1.778" layer="95"/>
+<pinref part="J5" gate="G$1" pin="4"/>
 </segment>
 <segment>
@@
 <label x="-167.64" y="-20.32" size="1.778" layer="95" rot="R180" xref="yes"/>
 </segment>
-<segment>
-<wire x1="-266.7" y1="63.5" x2="-246.38" y2="63.5" width="0.1524" layer="91"/>
-<label x="-261.62" y="63.5" size="1.778" layer="95"/>
-<pinref part="J5" gate="G$1" pin="5"/>
-</segment>
-</net>
-<net name="HALL_2_IN" class="0">
-<segment>
-<wire x1="-266.7" y1="60.96" x2="-246.38" y2="60.96" width="0.1524" layer="91"/>
-<label x="-261.62" y="60.96" size="1.778" layer="95"/>
-<pinref part="J5" gate="G$1" pin="4"/>
-</segment>
 </net>
 <net name="HALL_1_OUT" class="0">
@@
 </segment>
 <segment>
+<pinref part="U2" gate="A" pin="PB7"/>
+<wire x1="-5.08" y1="25.4" x2="12.7" y2="25.4" width="0.1524" layer="91"/>
+<label x="-2.54" y="25.4" size="1.778" layer="95"/>
+</segment>
+</net>
+<net name="HALL_2_OUT" class="0">
+<segment>
+<pinref part="U2" gate="A" pin="PB6"/>
+<wire x1="-5.08" y1="22.86" x2="12.7" y2="22.86" width="0.1524" layer="91"/>
+<label x="-2.54" y="22.86" size="1.778" layer="95"/>
+</segment>
+<segment>
 <pinref part="R10" gate="G$1" pin="2"/>
 <wire x1="-144.78" y1="15.24" x2="-142.24" y2="15.24" width="0.1524" layer="91"/>
@@
 <label x="-132.08" y="15.24" size="1.778" layer="95" xref="yes"/>
 </segment>
+</net>
+<net name="HALL_3_OUT" class="0">
+<segment>
+<pinref part="U2" gate="A" pin="PC11"/>
+<wire x1="-5.08" y1="7.62" x2="12.7" y2="7.62" width="0.1524" layer="91"/>
+<label x="-2.54" y="7.62" size="1.778" layer="95"/>
+</segment>
 <segment>
 <pinref part="R11" gate="G$1" pin="2"/>
@@
 <label x="-132.08" y="-20.32" size="1.778" layer="95" xref="yes"/>
 </segment>
-<segment>
-<pinref part="U2" gate="A" pin="PB7"/>
-<wire x1="-5.08" y1="25.4" x2="12.7" y2="25.4" width="0.1524" layer="91"/>
-<label x="-2.54" y="25.4" size="1.778" layer="95"/>
-</segment>
-</net>
-<net name="HALL_2_OUT" class="0">
-<segment>
-<pinref part="U2" gate="A" pin="PB6"/>
-<wire x1="-5.08" y1="22.86" x2="12.7" y2="22.86" width="0.1524" layer="91"/>
-<label x="-2.54" y="22.86" size="1.778" layer="95"/>
-</segment>
-</net>
-<net name="HALL_3_OUT" class="0">
-<segment>
-<pinref part="U2" gate="A" pin="PC11"/>
-<wire x1="-5.08" y1="7.62" x2="12.7" y2="7.62" width="0.1524" layer="91"/>
-<label x="-2.54" y="7.62" size="1.778" layer="95"/>
-</segment>
 </net>
 <net name="EN_GATE" class="0">
@@
 </net>
 <net name="SENS1" class="0">
-<segment>
-<wire x1="53.34" y1="7.62" x2="63.5" y2="7.62" width="0.1524" layer="91"/>
-<label x="53.34" y="7.62" size="1.778" layer="95"/>
-</segment>
 <segment>
 <pinref part="U2" gate="A" pin="PA2"/>
@@
 <net name="SENS2" class="0">
 <segment>
-<wire x1="53.34" y1="5.08" x2="63.5" y2="5.08" width="0.1524" layer="91"/>
-<label x="53.34" y="5.08" size="1.778" layer="95"/>
-</segment>
-<segment>
 <pinref part="U2" gate="A" pin="PA1"/>
 <wire x1="-55.88" y1="2.54" x2="-66.04" y2="2.54" width="0.1524" layer="91"/>
@@
 <net name="SENS3" class="0">
 <segment>
-<wire x1="53.34" y1="2.54" x2="63.5" y2="2.54" width="0.1524" layer="91"/>
-<label x="53.34" y="2.54" size="1.778" layer="95"/>
-</segment>
-<segment>
 <pinref part="U2" gate="A" pin="PA0-WKUP"/>
 <wire x1="-55.88" y1="5.08" x2="-66.04" y2="5.08" width="0.1524" layer="91"/>
@@
 <net name="FAULT" class="0">
 <segment>
-<wire x1="53.34" y1="-2.54" x2="63.5" y2="-2.54" width="0.1524" layer="91"/>
-<label x="53.34" y="-2.54" size="1.778" layer="95"/>
+<wire x1="53.34" y1="7.62" x2="63.5" y2="7.62" width="0.1524" layer="91"/>
+<label x="53.34" y="7.62" size="1.778" layer="95"/>
 </segment>
 <segment>
@@
 <net name="BR_SO1" class="0">
 <segment>
-<wire x1="53.34" y1="-7.62" x2="63.5" y2="-7.62" width="0.1524" layer="91"/>
-<label x="53.34" y="-7.62" size="1.778" layer="95"/>
+<wire x1="53.34" y1="2.54" x2="63.5" y2="2.54" width="0.1524" layer="91"/>
+<label x="53.34" y="2.54" size="1.778" layer="95"/>
 </segment>
 <segment>
@@
 <net name="BR_SO2" class="0">
 <segment>
-<wire x1="53.34" y1="-10.16" x2="63.5" y2="-10.16" width="0.1524" layer="91"/>
-<label x="53.34" y="-10.16" size="1.778" layer="95"/>
+<wire x1="53.34" y1="0" x2="63.5" y2="0" width="0.1524" layer="91"/>
+<label x="53.34" y="0" size="1.778" layer="95"/>
 </segment>
 <segment>
@@
 <net name="DC_CAL" class="0">
 <segment>
-<wire x1="53.34" y1="-12.7" x2="63.5" y2="-12.7" width="0.1524" layer="91"/>
-<label x="53.34" y="-12.7" size="1.778" layer="95"/>
-</segment>
-<segment>
+<wire x1="53.34" y1="-2.54" x2="63.5" y2="-2.54" width="0.1524" layer="91"/>
+<label x="53.34" y="-2.54" size="1.778" layer="95"/>
+</segment>
+<segment>

Commit message: stm32 module progress
Other:
- note added: "NEED TO CONNECT?????????????"
Changed lines of the file:
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@@
 <text x="-218.44" y="-30.48" size="1.778" layer="97" rot="R90">60V - 0V V_Batt</text>
 <text x="-447.04" y="185.42" size="1.778" layer="97">r35,36</text>
+<text x="-20.32" y="76.2" size="1.778" layer="91">NEED TO CONNECT?????????????</text>
 </plain>
 <instances>
